Commit message: modified the pkg to bringup imu_link and imu nodes

File: minibot_description/urdf/minibot.urdf.xacro (robot description, xacro)
@@ -121,4 +121,24 @@
             <origin xyz="0.02 0 0" rpy="0 0 0"/>
         </joint>
+        <!-- added by 0907smko@gmail.com -->
+        <!-- IMU Link -->
+		<link name="${prefix}imu_link">
+			<inertial>
+				<mass value="0.01"/>
+				<origin xyz="0 0 0" rpy="0 0 0"/>
+				<inertia ixx="0.00001" ixy="0.0" ixz="0.0" iyy="0.00001" iyz="0.0" izz="0.00001"/>
+			</inertial>
+			<collision>
+				<origin xyz="0 0 0" rpy="0 0 0"/>
+				<geometry>
+					<cylinder length="0.02" radius="0.01"/>
+				</geometry>
+			</collision>
+		</link>
+		<joint name="${prefix}imu_joint" type="fixed">
+			<parent link="${prefix}base_link"/>
+			<child link="${prefix}imu_link"/>
+			<origin xyz="0.1 0 0.1" rpy="0 0 0"/>
+		</joint>
     </xacro:macro>
 </robot>
